File: hardware/transverter_controller_test/transverter_controller_test.kicad_sch (KiCad schematic)
At the start: 46 parts, among them J1 USB_C_Receptacle_USB2.0, J2 Conn_01x04_Female, J3 Conn_01x05_Male, J4 Conn_01x05_Male, Q1 Si7141DP, Q2 SI1539CDL-T1-GE3, Q3 Si7141DP, Q4 SI1539CDL-T1-GE3, Q5 Si7141DP, Q6 SI1539CDL-T1-GE3, SW1 SW_Push, U1 MKL26Z64VFT4, U2 MKL02Z32VFG4, U3 INA237, U4 INA237, U5 INA237, U6 24LC64FT-I/MNY, Y1 830108178109

Commit message: v1 transverter interface complete
Parts:
- removed C11, C8, C9: 100n, Capacitor_SMD:C_0402_1005Metric, symbol Device:C
- removed C4: DNF, Capacitor_SMD:C_0603_1608Metric, symbol Device:C
- removed J2: Conn_01x04_Female, Connector_PinSocket_2.54mm:PinSocket_1x04_P2.54mm_Horizontal, symbol Connector:Conn_01x04_Female
- removed J3, J4: Conn_01x05_Male, Connector_WUT:Weidmuller_SL3.5-5-90G, symbol Connector:Conn_01x05_Male
- removed Q1, Q3, Q5: Si7141DP, Package_SO:PowerPAK_SO-8_Single, symbol Transistor_FET:Si7141DP
- removed Q2, Q4, Q6: SI1539CDL-T1-GE3, Package_TO_SOT_SMD:SOT-363_SC-70-6, symbol FET_WUT:SI1539CDL-T1-GE3
- removed SW1: SW_Push, Button_Switch_SMD:SW_Push_SPST_NO_Alps_SKRK, symbol Switch:SW_Push
- removed U2: MKL02Z32VFG4, Package_DFN_QFN:QFN-16-1EP_3x3mm_P0.5mm_EP1.9x1.9mm, symbol MCU_NXP_Kinetis:MKL02Z32VFG4
- removed U3, U4, U5: INA237, Package_SO:VSSOP-10_3x3mm_P0.5mm, symbol IC_WUT:INA237
- removed U6: 24LC64FT-I/MNY, Package_DFN_QFN:DFN-8-1EP_3x2mm_P0.5mm_EP1.36x1.46mm, symbol Memory_EEPROM:24LC64
- added C1: 100n, Capacitor_SMD:C_0402_1005Metric, symbol Device:C
- added C2: DNF, Capacitor_SMD:C_0402_1005Metric, symbol Device:C
- added H1, H2, H3: MountingHole_Pad, MountingHole:MountingHole_3.2mm_M3_Pad_Via, symbol Mechanical:MountingHole_Pad
- added J1, J4: CNC Tech 3020-10-0200-00‎, Connector_WUT:Header_CNC-Tech_3020-10-0200-00_2x5_TH_RA, symbol Connector_Generic:Conn_02x05_Odd_Even
- added J3: Conn_01x03_Male, Connector_PinHeader_2.54mm:PinHeader_1x03_P2.54mm_Vertical, symbol Connector:Conn_01x03_Male
- added JP1: SolderJumper_2_Open, Jumper:SolderJumper-2_P1.3mm_Open_RoundedPad1.0x1.5mm, symbol Jumper:SolderJumper_2_Open
- added LD1: Kingbright_WP130WCP_2EGW, LED_WUT:Kingbright_WP130WCP_2EGW, symbol LED_WUT:Kingbright_WP130WCP_2EGW
- added M1: Logo_10mmx10mm, Misc_WUT:Logo_10mmx10mm, symbol Misc_WUT:Logo_10mmx10mm
- added Q1, Q2: DMN62D0U-13, Package_TO_SOT_SMD:SOT-23, symbol Device:Q_NMOS_GSD
- added U1: PCT2075D, Package_SO:SO-8_3.9x4.9mm_P1.27mm, symbol Sensor_Temperature:PCT2075D
- added U2: 24LC024-I/SN, Package_SO:SO-8_3.9x4.9mm_P1.27mm, symbol Memory_EEPROM:24LC02
- added U4: MAX3483ESA+, Package_SO:SO-8_3.9x4.9mm_P1.27mm, symbol Interface_UART:MAX3483
- R10: value 10k -> DNF; footprint Resistor_SMD:R_0402_1005Metric -> Resistor_SMD:R_0603_1608Metric
- R11, R12, R13, R14, R7: value 10k -> 1k
- R3: value 0R1 -> 10k; footprint Resistor_SMD:R_2512_6332Metric -> Resistor_SMD:R_0402_1005Metric
- R4, R5: value 0R1 -> 4k7; footprint Resistor_SMD:R_2512_6332Metric -> Resistor_SMD:R_0402_1005Metric
- renumbered C1 to C3, C2 to C4, C3 to C5, C5 to C6, C6 to C7, C12 to C8, C7 to C9, FB2 to FB1, FB1 to FB2, J1 to J2, U1 to U3
Connections:
- net +12V is gone; now on net +3V3: R3.1
- net +28V is gone; now on net +3V3: R4.1
- net +48V is gone; now on net +3V3: R5.1
- net D20 is gone; now on net LED_ERROR: U3.46 (PTD5)
- net D21 is gone; now on net LED_STATUS: U3.47 (PTD6/LLWU_P15)
- net D5 is gone; now on net LED_RX: U3.48 (PTD7)
- net D6 is gone; now on net LED_TX: U3.45 (PTD4/LLWU_P14)
- net D8 is gone; now on an unnamed net: U3.44 (PTD3)
- net ~28V_ALERT is gone; now on net WP: R7.2
- net +3V3: now also C3.1, C4.1, C5.1, C6.1, C7.1, U3.1 (VDD), U3.22 (VDD), U3.6 (VREGIN), U3.9 (VDDA), C1.1, U1.8 (VCC), U2.8 (VCC), U4.8 (VCC); no longer R8.1
- net GND: now also R8.2, R9.2, C1.2, C2.2, H1.1, H2.1, H3.1, J1.2 (Pin_2), J3.3 (Pin_3), J4.10 (Pin_10), JP1.2 (B), LD1.2, LD1.5, Q1.2 (S), Q2.2 (S), U1.4 (GND), U1.5 (A2), U1.6 (A1), U1.7 (A0), U2.1 (A0), U2.2 (A1), U2.3 (A2), U2.4 (GND), U4.5 (GND); no longer R10.2, R12.2, R14.2
- net PTA0: now also J1.10 (Pin_10)
- net PTA3: now also J1.9 (Pin_9)
- net RESET_B: now also R3.2, C2.1, J1.8 (Pin_8)
- net SCL: now also R4.2, J1.6 (Pin_6), U1.2 (SCL), U2.6 (SCL)
- net SDA: now also R5.2, J1.5 (Pin_5), U1.1 (SDA), U2.5 (SDA)
- net LED_STATUS: now reaches R14.1
- net at R13.2: now also LD1.4
- net LED_TX: now reaches R11.1
- net LED_TX: no longer R4.2
- net at R11.2: now also LD1.1
- net LED_RX: now reaches R12.1
- net at R9.1: now also Q2.1 (G); no longer R3.2
- net at J2.A7 (D-), J2.B7 (D-): now also R1.1; no longer R2.1
- net D_N: now reaches R2.2
- net D_N: now also U3.3 (USB0_DP); no longer U3.4 (USB0_DM)
- net at J2.A6 (D+), J2.B6 (D+): now also R2.1; no longer R1.1
- net D_P: now reaches R1.2
- net D_P: now also U3.4 (USB0_DM); no longer U3.3 (USB0_DP)
- net LED_ERROR: now reaches R13.1
- net LED_ERROR: no longer R5.2
- net RS485_B: now reaches R10.1
- net RS485_B: now also J1.4 (Pin_4), U4.7 (B)
- net D0 renamed RX
- net RX: now also U4.1 (RO)
- net D1 renamed TX
- net TX: now also U4.4 (DI)
- net D10 renamed SPARE_6
- net SPARE_6: now also J4.6 (Pin_6)
- net D11 renamed SPARE_4
- net SPARE_4: now also J4.4 (Pin_4)
- net D12 renamed SPARE_3
- net SPARE_3: now also J4.3 (Pin_3)
- net D13 renamed SPARE_5
- net SPARE_5: now also J4.5 (Pin_5)
- net D14 renamed SPARE_1
- net SPARE_1: now also J4.1 (Pin_1)
- net D15 renamed ~R~/W
- net ~R~/W: now also U4.2 (~RE), U4.3 (DE)
- net D16 renamed WP
- net WP: now also J1.7 (Pin_7), JP1.1 (A), U2.7 (WP)
- net D17 renamed ~OVERTEMP
- net ~OVERTEMP: now also R6.2, U1.3 (OS)
- net D2 renamed SPARE_2
- net SPARE_2: now also J4.2 (Pin_2)
- net D22 renamed SPARE_9
- net SPARE_9: now also J4.9 (Pin_9)
- net D23 renamed SPARE_8
- net SPARE_8: now also J4.8 (Pin_8)
- net D26: no longer names the net of U3.14 (PTE30)
- net D3: no longer names the net of U3.18 (PTA1)
- net D4: no longer names the net of U3.19 (PTA2)
- net D7: no longer names the net of U3.43 (PTD2)
- net D7: now also R8.1, Q1.1 (G)
- net D9 renamed SPARE_7
- net SPARE_7: now also J4.7 (Pin_7)
- removed net ~12V_ALERT: R6.2, R8.2
- new net: LD1.3, R12.2
- new net: LD1.6, R14.2
- new net: FB1.2, J1.1 (Pin_1)
- new net: J3.1 (Pin_1), Q1.3 (D)
- new net: J3.2 (Pin_2), Q2.3 (D)
- new net RS485_A: J1.3 (Pin_3), R10.2, U4.6 (A)
- no-connect marks 29 -> 15
Other:
- note added: "D0"
- note added: "D1"
- note added: "D10"
- note added: "D11"
- note added: "D12"
- note added: "D13"
- note added: "D14"
- note added: "D15"
- note added: "D16"
- note added: "D17"
- note added: "D2"
- note added: "D20"
- note added: "D21"
- note added: "D22"
- note added: "D23"
- note added: "D26"
- note added: "D3"
- note added: "D4"
- note added: "D5"
- note added: "D6"
- note added: "D7"
- note added: "D8"
- note added: "D9"
- note added: "I2C Address = 0x48"
- note added: "I2C Address = 0x50"
- note added: "Short jumper to allow EEPROM programming"
- moved on the sheet: C3, C4, C5, C6, C7, C8, C9, FB1, FB2, J2, R1, R2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
