File: hardware/rs485_test/transverter.kicad_sch (KiCad schematic)
At the start: 5 parts, among them J1 CNC Tech 3020-10-0100-00‎, J2 Conn_01x02_Male, U1 24LC024-I/SN

Commit message: Added RS485 driver and AXI GPIO for read/write
Parts:
- renumbered C1 to C6, J1 to J10, J2 to J11, R1 to R6, U1 to U6
Changed lines of the file:
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@@
   (symbol (lib_id "power:+3V3") (at 105.41 85.09 0)
     (in_bom yes) (on_board yes) (fields_autoplaced)
-    (property "Reference" "#PWR01" (id 0) (at 105.41 88.9 0)
+    (property "Reference" "#PWR037" (id 0) (at 105.41 88.9 0)
       (effects (font (size 1.27 1.27)) hide)
     )
@@
   (symbol (lib_id "power:+3.3V") (at 123.19 46.99 0)
     (in_bom yes) (on_board yes) (fields_autoplaced)
-    (property "Reference" "#PWR04" (id 0) (at 123.19 50.8 0)
+    (property "Reference" "#PWR040" (id 0) (at 123.19 50.8 0)
       (effects (font (size 1.27 1.27)) hide)
     )
@@
   (symbol (lib_id "power:+3.3V") (at 146.05 100.33 0)
     (in_bom yes) (on_board yes) (fields_autoplaced)
-    (property "Reference" "#PWR07" (id 0) (at 146.05 104.14 0)
+    (property "Reference" "#PWR043" (id 0) (at 146.05 104.14 0)
       (effects (font (size 1.27 1.27)) hide)
     )
@@
   (symbol (lib_id "power:GND") (at 109.22 96.52 0)
     (in_bom yes) (on_board yes) (fields_autoplaced)
-    (property "Reference" "#PWR02" (id 0) (at 109.22 102.87 0)
+    (property "Reference" "#PWR038" (id 0) (at 109.22 102.87 0)
       (effects (font (size 1.27 1.27)) hide)
     )
@@
   (symbol (lib_id "power:GND") (at 114.3 121.92 0)
     (in_bom yes) (on_board yes) (fields_autoplaced)
-    (property "Reference" "#PWR03" (id 0) (at 114.3 128.27 0)
+    (property "Reference" "#PWR039" (id 0) (at 114.3 128.27 0)
       (effects (font (size 1.27 1.27)) hide)
     )
@@
   (symbol (lib_id "power:GND") (at 127 121.92 0)
     (in_bom yes) (on_board yes) (fields_autoplaced)
-    (property "Reference" "#PWR05" (id 0) (at 127 128.27 0)
+    (property "Reference" "#PWR041" (id 0) (at 127 128.27 0)
       (effects (font (size 1.27 1.27)) hide)
     )
@@
   (symbol (lib_id "power:GND") (at 139.7 63.5 0)
     (in_bom yes) (on_board yes) (fields_autoplaced)
-    (property "Reference" "#PWR06" (id 0) (at 139.7 69.85 0)
+    (property "Reference" "#PWR042" (id 0) (at 139.7 69.85 0)
       (effects (font (size 1.27 1.27)) hide)
     )
@@
   (symbol (lib_id "power:GND") (at 146.05 123.19 0)
     (in_bom yes) (on_board yes) (fields_autoplaced)
-    (property "Reference" "#PWR08" (id 0) (at 146.05 129.54 0)
+    (property "Reference" "#PWR044" (id 0) (at 146.05 129.54 0)
       (effects (font (size 1.27 1.27)) hide)
     )
@@
   (symbol (lib_id "Connector:Conn_01x02_Male") (at 153.67 118.11 0) (mirror y)
     (in_bom yes) (on_board yes) (fields_autoplaced)
-    (property "Reference" "J2" (id 0) (at 154.94 118.7449 0)
+    (property "Reference" "J11" (id 0) (at 154.94 118.7449 0)
       (effects (font (size 1.27 1.27)) (justify right))
     )
@@
   (symbol (lib_id "Device:R") (at 146.05 106.68 0)
     (in_bom yes) (on_board yes) (fields_autoplaced)
-    (property "Reference" "R1" (id 0) (at 148.59 106.0449 0)
+    (property "Reference" "R6" (id 0) (at 148.59 106.0449 0)
       (effects (font (size 1.27 1.27)) (justify left))
     )
@@
   (symbol (lib_id "Device:C") (at 109.22 91.44 0)
     (in_bom yes) (on_board yes) (fields_autoplaced)
-    (property "Reference" "C1" (id 0) (at 113.03 90.8049 0)
+    (property "Reference" "C6" (id 0) (at 113.03 90.8049 0)
       (effects (font (size 1.27 1.27)) (justify left))
     )
@@
   (symbol (lib_id "Connector_Generic:Conn_02x05_Odd_Even") (at 130.81 55.88 0)
     (in_bom yes) (on_board yes)
-    (property "Reference" "J1" (id 0) (at 130.81 46.99 0))
+    (property "Reference" "J10" (id 0) (at 130.81 46.99 0))
     (property "Value" "CNC Tech 3020-10-0100-00‎ " (id 1) (at 149.86 46.99 0))
     (property "Footprint" "Connector_PinHeader_2.54mm:PinHeader_2x05_P2.54mm_Vertical" (id 2) (at 130.81 55.88 0)
@@
   (symbol (lib_id "Memory_EEPROM:24LC02") (at 127 110.49 0)
     (in_bom yes) (on_board yes)
-    (property "Reference" "U1" (id 0) (at 120.65 104.14 0))
+    (property "Reference" "U6" (id 0) (at 120.65 104.14 0))
     (property "Value" "24LC024-I/SN" (id 1) (at 135.89 118.11 0))
     (property "Footprint" "Package_SO:SO-8_3.9x4.9mm_P1.27mm" (id 2) (at 127 110.49 0)
