File: hardware/RF_front_end/_autosave-RF_front_end.kicad_sch (KiCad schematic)
At the start: 14 parts, among them J1 Conn_Coaxial, J2 Conn_Coaxial, Q1 SI1539CDL-T1-GE3

Commit message: More work on front end
Parts:
- removed C6: 100n, Capacitor_SMD:C_0402_1005Metric, symbol Device:C
Changed lines of the file:
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@@
     (stroke (width 0) (type solid) (color 0 0 0 0))
   )
-  (wire (pts (xy 191.77 86.36) (xy 209.55 86.36))
-    (stroke (width 0) (type solid) (color 0 0 0 0))
-  )
-  (wire (pts (xy 191.77 113.03) (xy 196.85 113.03))
+  (wire (pts (xy 191.77 113.03) (xy 205.74 113.03))
     (stroke (width 0) (type solid) (color 0 0 0 0))
   )
@@
     (stroke (width 0) (type solid) (color 0 0 0 0))
   )
-  (wire (pts (xy 205.74 91.44) (xy 205.74 113.03))
-    (stroke (width 0) (type solid) (color 0 0 0 0))
-  )
-  (wire (pts (xy 205.74 113.03) (xy 204.47 113.03))
+  (wire (pts (xy 198.12 86.36) (xy 191.77 86.36))
+    (stroke (width 0) (type solid) (color 0 0 0 0))
+  )
+  (wire (pts (xy 198.12 91.44) (xy 198.12 86.36))
+    (stroke (width 0) (type solid) (color 0 0 0 0))
+  )
+  (wire (pts (xy 205.74 86.36) (xy 205.74 113.03))
     (stroke (width 0) (type solid) (color 0 0 0 0))
   )
@@
     (stroke (width 0) (type solid) (color 0 0 0 0))
   )
-  (wire (pts (xy 209.55 91.44) (xy 205.74 91.44))
+  (wire (pts (xy 209.55 86.36) (xy 205.74 86.36))
+    (stroke (width 0) (type solid) (color 0 0 0 0))
+  )
+  (wire (pts (xy 209.55 91.44) (xy 198.12 91.44))
     (stroke (width 0) (type solid) (color 0 0 0 0))
   )
@@
     )
     (property "Datasheet" "~" (id 3) (at 157.48 113.03 0)
-      (effects (font (size 1.27 1.27)) hide)
-    )
-    (pin "1")
-    (pin "2")
-  )
-  (symbol (lib_id "Device:C") (at 200.66 113.03 90) (unit 1)
-    (in_bom yes) (on_board yes) (fields_autoplaced)
-    (property "Reference" "C6" (id 0) (at 200.66 106.68 90))
-    (property "Value" "100n" (id 1) (at 200.66 109.22 90))
-    (property "Footprint" "Capacitor_SMD:C_0402_1005Metric" (id 2) (at 204.47 112.0648 0)
-      (effects (font (size 1.27 1.27)) hide)
-    )
-    (property "Datasheet" "~" (id 3) (at 200.66 113.03 0)
       (effects (font (size 1.27 1.27)) hide)
     )
@@
       (reference "C5") (unit 1) (value "100n") (footprint "Capacitor_SMD:C_0402_1005Metric")
     )
-    (path "/0515e187-b57b-4ba9-bc23-814282bbbd25"
-      (reference "C6") (unit 1) (value "100n") (footprint "Capacitor_SMD:C_0402_1005Metric")
-    )
     (path "/38b4da4d-24fe-4395-b6f1-64713392f61c"
       (reference "C7") (unit 1) (value "100n") (footprint "Capacitor_SMD:C_0402_1005Metric")
@@
       (reference "R3") (unit 1) (value "10k") (footprint "Resistor_SMD:R_0402_1005Metric")
     )
-    (path "/252479cc-af31-4b51-bb44-c6eb506168c7/8b8549af-748c-44eb-9f1d-2220742f596c"
-      (reference "R4") (unit 1) (value "0") (footprint "Resistor_SMD:R_0402_1005Metric")
-    )
-    (path "/dd3cae6a-0b6b-477f-86d5-aef1dbba5c15/8b8549af-748c-44eb-9f1d-2220742f596c"
-      (reference "R5") (unit 1) (value "0") (footprint "Resistor_SMD:R_0402_1005Metric")
-    )
-    (path "/2a98e36a-32f1-4eb4-9672-185a87e5884e/8b8549af-748c-44eb-9f1d-2220742f596c"
-      (reference "R6") (unit 1) (value "0") (footprint "Resistor_SMD:R_0402_1005Metric")
-    )
     (path "/252479cc-af31-4b51-bb44-c6eb506168c7/331d1669-b4d4-4493-a2f8-15ec1ffd0dcb"
