File: hardware/RF_front_end/RF_front_end.kicad_sch (KiCad schematic)
At the start: 14 parts, among them J1 Conn_Coaxial, J2 Conn_Coaxial, Q1 SI1539CDL-T1-GE3

Commit message: Finished front end
Parts:
- removed C6: 100n, Capacitor_SMD:C_0402_1005Metric, symbol Device:C
- added C3: 10u, Capacitor_SMD:C_0603_1608Metric, symbol Device:C
- added C5: 1u, Capacitor_SMD:C_0402_1005Metric, symbol Device:C
- added D1, D2, D3, D4, D5: LED, LED_SMD:LED_0603_1608Metric, symbol Device:LED
- added FB1: FerriteBead_Small, Inductor_SMD:L_0603_1608Metric, symbol Device:FerriteBead_Small
- added J2: Conn_01x07_Male, Connector_PinHeader_2.54mm:PinHeader_1x07_P2.54mm_Vertical, symbol Connector:Conn_01x07_Male
- added M1: Logo_10mmx10mm, Misc_WUT:Logo_10mmx10mm, symbol Misc_WUT:Logo_10mmx10mm
- added R1, R2, R3, R4, R5: 1k, Resistor_SMD:R_0402_1005Metric, symbol Device:R
- added R10, R6, R7, R8, R9: 100, Resistor_SMD:R_0402_1005Metric, symbol Device:R
- renumbered C3 to C4, C4 to C6, C5 to C7, C7 to C8, J2 to J3, R1 to R11, R2 to R12, R3 to R13
Connections:
- net +3V3: now also C3.1, C5.1, D1.2 (A), D2.2 (A), D3.2 (A), D4.2 (A), D5.2 (A), FB1.2
- net ATT_EN: now also R8.2
- net GND: now also C3.2, C5.2, J2.2 (Pin_2)
- new net: D3.1 (K), R3.1
- new net: J2.4 (Pin_4), R2.2, R9.1
- new net: D5.1 (K), R5.1
- new net: D2.1 (K), R2.1
- new net: D1.1 (K), R1.1
- new net: J2.3 (Pin_3), R1.2, R6.1
- new net: FB1.1, J2.1 (Pin_1)
- new net: J2.5 (Pin_5), R3.2, R7.1
- new net: J2.6 (Pin_6), R10.1, R4.2
- new net: J2.7 (Pin_7), R5.2, R8.1
- new net: D4.1 (K), R4.1
- new net ATT0: R6.2
- new net ATT1: R9.2
- new net ATT2: R7.2
- new net ATT3: R10.2
Other:
- sheet Adjustable Attenuator ports: added ATT0, ATT1, ATT2, ATT3; removed ATT
