File: hardware/RF_front_end/attenuator.kicad_sch (KiCad schematic)
At the start: 4 parts, among them U5 RFSA3413

Commit message: Finished front end
Parts:
- U5: footprint Package_DFN_QFN:QFN-16-1EP_3x3mm_P0.5mm_EP1.7x1.7mm_ThermalVias -> Package_DFN_QFN:QFN-16-1EP_3x3mm_P0.5mm_EP1.7x1.7mm
- renumbered C18 to C19, C19 to C20, FB5 to FB6
Changed lines of the file:
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@@
   (junction (at 162.56 106.68) (diameter 0.9144) (color 0 0 0 0))
   (junction (at 162.56 109.22) (diameter 0.9144) (color 0 0 0 0))
-  (bus_entry (at 125.73 91.44) (size 2.54 -2.54)
-    (stroke (width 0.1524) (type solid) (color 0 0 0 0))
-  )
-  (bus_entry (at 125.73 93.98) (size 2.54 -2.54)
-    (stroke (width 0.1524) (type solid) (color 0 0 0 0))
-  )
-  (bus_entry (at 125.73 96.52) (size 2.54 -2.54)
-    (stroke (width 0.1524) (type solid) (color 0 0 0 0))
-  )
-  (bus_entry (at 125.73 99.06) (size 2.54 -2.54)
-    (stroke (width 0.1524) (type solid) (color 0 0 0 0))
-  )
   (wire (pts (xy 118.11 50.8) (xy 118.11 46.99))
     (stroke (width 0) (type solid) (color 0 0 0 0))
@@
     (stroke (width 0) (type solid) (color 0 0 0 0))
   )
-  (bus (pts (xy 119.38 100.33) (xy 125.73 100.33))
-    (stroke (width 0) (type solid) (color 0 0 0 0))
-  )
-  (bus (pts (xy 125.73 91.44) (xy 125.73 100.33))
-    (stroke (width 0) (type solid) (color 0 0 0 0))
-  )
-  (label "ATT0" (at 129.54 88.9 0)
-    (effects (font (size 1.27 1.27)) (justify left bottom))
-  )
-  (label "ATT1" (at 129.54 91.44 0)
-    (effects (font (size 1.27 1.27)) (justify left bottom))
-  )
-  (label "ATT2" (at 129.54 93.98 0)
-    (effects (font (size 1.27 1.27)) (justify left bottom))
-  )
-  (label "ATT3" (at 129.54 96.52 0)
-    (effects (font (size 1.27 1.27)) (justify left bottom))
-  )
   (hierarchical_label "RFIN" (shape input) (at 119.38 83.82 180)
     (effects (font (size 1.27 1.27)) (justify right))
   )
-  (hierarchical_label "ATT" (shape input) (at 119.38 100.33 180)
+  (hierarchical_label "ATT0" (shape input) (at 128.27 88.9 180)
+    (effects (font (size 1.27 1.27)) (justify right))
+  )
+  (hierarchical_label "ATT1" (shape input) (at 128.27 91.44 180)
+    (effects (font (size 1.27 1.27)) (justify right))
+  )
+  (hierarchical_label "ATT2" (shape input) (at 128.27 93.98 180)
+    (effects (font (size 1.27 1.27)) (justify right))
+  )
+  (hierarchical_label "ATT3" (shape input) (at 128.27 96.52 180)
     (effects (font (size 1.27 1.27)) (justify right))
   )
@@
   (symbol (lib_id "power:+3.3V") (at 118.11 46.99 0) (unit 1)
     (in_bom yes) (on_board yes) (fields_autoplaced)
-    (property "Reference" "#PWR025" (id 0) (at 118.11 50.8 0)
+    (property "Reference" "#PWR029" (id 0) (at 118.11 50.8 0)
       (effects (font (size 1.27 1.27)) hide)
     )
@@
   (symbol (lib_id "power:GND") (at 134.62 63.5 0) (unit 1)
     (in_bom yes) (on_board yes) (fields_autoplaced)
-    (property "Reference" "#PWR026" (id 0) (at 134.62 69.85 0)
+    (property "Reference" "#PWR030" (id 0) (at 134.62 69.85 0)
       (effects (font (size 1.27 1.27)) hide)
     )
@@
   (symbol (lib_id "power:GND") (at 148.59 116.84 0) (unit 1)
     (in_bom yes) (on_board yes) (fields_autoplaced)
-    (property "Reference" "#PWR027" (id 0) (at 148.59 123.19 0)
+    (property "Reference" "#PWR031" (id 0) (at 148.59 123.19 0)
       (effects (font (size 1.27 1.27)) hide)
     )
@@
   (symbol (lib_id "power:GND") (at 162.56 111.76 0) (unit 1)
     (in_bom yes) (on_board yes) (fields_autoplaced)
-    (property "Reference" "#PWR028" (id 0) (at 162.56 118.11 0)
+    (property "Reference" "#PWR032" (id 0) (at 162.56 118.11 0)
       (effects (font (size 1.27 1.27)) hide)
     )
@@
   (symbol (lib_id "Device:FerriteBead_Small") (at 129.54 50.8 90) (unit 1)
     (in_bom yes) (on_board yes) (fields_autoplaced)
-    (property "Reference" "FB5" (id 0) (at 129.54 45.72 90))
+    (property "Reference" "FB6" (id 0) (at 129.54 45.72 90))
     (property "Value" "FerriteBead_Small" (id 1) (at 129.54 48.26 90))
     (property "Footprint" "Inductor_SMD:L_0402_1005Metric" (id 2) (at 129.54 52.578 90)
@@
   (symbol (lib_id "Device:C") (at 134.62 57.15 0) (unit 1)
     (in_bom yes) (on_board yes) (fields_autoplaced)
-    (property "Reference" "C18" (id 0) (at 138.43 56.5149 0)
+    (property "Reference" "C19" (id 0) (at 138.43 56.5149 0)
       (effects (font (size 1.27 1.27)) (justify left))
     )
@@
   (symbol (lib_id "Device:C") (at 171.45 83.82 90) (unit 1)
     (in_bom yes) (on_board yes) (fields_autoplaced)
-    (property "Reference" "C19" (id 0) (at 171.45 77.47 90))
+    (property "Reference" "C20" (id 0) (at 171.45 77.47 90))
     (property "Value" "100n" (id 1) (at 171.45 80.01 90))
     (property "Footprint" "Capacitor_SMD:C_0402_1005Metric" (id 2) (at 175.26 82.8548 0)
@@
     (pin "2")
   )
-  (symbol (lib_id "RF_WUT:RFSA3413") (at 148.59 83.82 0) (unit 1)
+  (symbol (lib_id "RF_WUT:RFSA3413") (at 148.59 83.82 0)
     (in_bom yes) (on_board yes)
     (property "Reference" "U5" (id 0) (at 151.13 77.47 0))
     (property "Value" "RFSA3413" (id 1) (at 154.94 113.03 0))
-    (property "Footprint" "Package_DFN_QFN:QFN-16-1EP_3x3mm_P0.5mm_EP1.7x1.7mm_ThermalVias" (id 2) (at 148.59 83.82 0)
-      (effects (font (size 1.27 1.27)) hide)
-    )
+    (property "Footprint" "Package_DFN_QFN:QFN-16-1EP_3x3mm_P0.5mm_EP1.7x1.7mm" (id 2) (at 148.59 83.82 0)
+      (effects (font (size 1.27 1.27)) hide)
+    )
