File: hardware/RF_front_end/bpf.kicad_sch (KiCad schematic)
At the start: 14 parts

Commit message: Finished front end
Parts:
- renumbered C24 to C25, C25 to C26, C26 to C27, C27 to C28, C28 to C29, C29 to C30, C30 to C31, C31 to C32, C32 to C33, C33 to C34, C34 to C35
Changed lines of the file:
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@@
   (symbol (lib_id "power:GND") (at 93.98 106.68 0) (unit 1)
     (in_bom yes) (on_board yes) (fields_autoplaced)
-    (property "Reference" "#PWR035" (id 0) (at 93.98 113.03 0)
+    (property "Reference" "#PWR039" (id 0) (at 93.98 113.03 0)
       (effects (font (size 1.27 1.27)) hide)
     )
@@
   (symbol (lib_id "power:GND") (at 104.14 106.68 0) (unit 1)
     (in_bom yes) (on_board yes) (fields_autoplaced)
-    (property "Reference" "#PWR036" (id 0) (at 104.14 113.03 0)
+    (property "Reference" "#PWR040" (id 0) (at 104.14 113.03 0)
       (effects (font (size 1.27 1.27)) hide)
     )
@@
   (symbol (lib_id "power:GND") (at 124.46 106.68 0) (unit 1)
     (in_bom yes) (on_board yes) (fields_autoplaced)
-    (property "Reference" "#PWR037" (id 0) (at 124.46 113.03 0)
+    (property "Reference" "#PWR041" (id 0) (at 124.46 113.03 0)
       (effects (font (size 1.27 1.27)) hide)
     )
@@
   (symbol (lib_id "power:GND") (at 134.62 106.68 0) (unit 1)
     (in_bom yes) (on_board yes) (fields_autoplaced)
-    (property "Reference" "#PWR038" (id 0) (at 134.62 113.03 0)
+    (property "Reference" "#PWR042" (id 0) (at 134.62 113.03 0)
       (effects (font (size 1.27 1.27)) hide)
     )
@@
   (symbol (lib_id "power:GND") (at 154.94 106.68 0) (unit 1)
     (in_bom yes) (on_board yes) (fields_autoplaced)
-    (property "Reference" "#PWR039" (id 0) (at 154.94 113.03 0)
+    (property "Reference" "#PWR043" (id 0) (at 154.94 113.03 0)
       (effects (font (size 1.27 1.27)) hide)
     )
@@
   (symbol (lib_id "power:GND") (at 165.1 106.68 0) (unit 1)
     (in_bom yes) (on_board yes) (fields_autoplaced)
-    (property "Reference" "#PWR040" (id 0) (at 165.1 113.03 0)
+    (property "Reference" "#PWR044" (id 0) (at 165.1 113.03 0)
       (effects (font (size 1.27 1.27)) hide)
     )
@@
   (symbol (lib_id "power:GND") (at 185.42 106.68 0) (unit 1)
     (in_bom yes) (on_board yes) (fields_autoplaced)
-    (property "Reference" "#PWR041" (id 0) (at 185.42 113.03 0)
+    (property "Reference" "#PWR045" (id 0) (at 185.42 113.03 0)
       (effects (font (size 1.27 1.27)) hide)
     )
@@
   (symbol (lib_id "power:GND") (at 195.58 106.68 0) (unit 1)
     (in_bom yes) (on_board yes) (fields_autoplaced)
-    (property "Reference" "#PWR042" (id 0) (at 195.58 113.03 0)
+    (property "Reference" "#PWR046" (id 0) (at 195.58 113.03 0)
       (effects (font (size 1.27 1.27)) hide)
     )
@@
   (symbol (lib_id "Device:C") (at 93.98 100.33 0) (unit 1)
     (in_bom yes) (on_board yes) (fields_autoplaced)
-    (property "Reference" "C24" (id 0) (at 97.79 99.6949 0)
+    (property "Reference" "C25" (id 0) (at 97.79 99.6949 0)
       (effects (font (size 1.27 1.27)) (justify left))
     )
@@
   (symbol (lib_id "Device:C") (at 104.14 100.33 0) (unit 1)
     (in_bom yes) (on_board yes) (fields_autoplaced)
-    (property "Reference" "C25" (id 0) (at 107.95 99.6949 0)
+    (property "Reference" "C26" (id 0) (at 107.95 99.6949 0)
       (effects (font (size 1.27 1.27)) (justify left))
     )
@@
   (symbol (lib_id "Device:C") (at 115.57 83.82 90) (unit 1)
     (in_bom yes) (on_board yes) (fields_autoplaced)
-    (property "Reference" "C26" (id 0) (at 115.57 77.47 90))
+    (property "Reference" "C27" (id 0) (at 115.57 77.47 90))
     (property "Value" "C" (id 1) (at 115.57 80.01 90))
     (property "Footprint" "Capacitor_SMD:C_0402_1005Metric" (id 2) (at 119.38 82.8548 0)
@@
   (symbol (lib_id "Device:C") (at 124.46 100.33 0) (unit 1)
     (in_bom yes) (on_board yes) (fields_autoplaced)
-    (property "Reference" "C27" (id 0) (at 128.27 99.6949 0)
+    (property "Reference" "C28" (id 0) (at 128.27 99.6949 0)
       (effects (font (size 1.27 1.27)) (justify left))
     )
@@
   (symbol (lib_id "Device:C") (at 134.62 100.33 0) (unit 1)
     (in_bom yes) (on_board yes) (fields_autoplaced)
-    (property "Reference" "C28" (id 0) (at 138.43 99.6949 0)
+    (property "Reference" "C29" (id 0) (at 138.43 99.6949 0)
       (effects (font (size 1.27 1.27)) (justify left))
     )
@@
   (symbol (lib_id "Device:C") (at 146.05 83.82 90) (unit 1)
     (in_bom yes) (on_board yes) (fields_autoplaced)
-    (property "Reference" "C29" (id 0) (at 146.05 77.47 90))
+    (property "Reference" "C30" (id 0) (at 146.05 77.47 90))
     (property "Value" "C" (id 1) (at 146.05 80.01 90))
     (property "Footprint" "Capacitor_SMD:C_0402_1005Metric" (id 2) (at 149.86 82.8548 0)
@@
   (symbol (lib_id "Device:C") (at 154.94 100.33 0) (unit 1)
     (in_bom yes) (on_board yes) (fields_autoplaced)
-    (property "Reference" "C30" (id 0) (at 158.75 99.6949 0)
+    (property "Reference" "C31" (id 0) (at 158.75 99.6949 0)
       (effects (font (size 1.27 1.27)) (justify left))
     )
@@
   (symbol (lib_id "Device:C") (at 165.1 100.33 0) (unit 1)
     (in_bom yes) (on_board yes) (fields_autoplaced)
-    (property "Reference" "C31" (id 0) (at 168.91 99.6949 0)
+    (property "Reference" "C32" (id 0) (at 168.91 99.6949 0)
       (effects (font (size 1.27 1.27)) (justify left))
     )
@@
   (symbol (lib_id "Device:C") (at 176.53 83.82 90) (unit 1)
     (in_bom yes) (on_board yes) (fields_autoplaced)
-    (property "Reference" "C32" (id 0) (at 176.53 77.47 90))
+    (property "Reference" "C33" (id 0) (at 176.53 77.47 90))
     (property "Value" "C" (id 1) (at 176.53 80.01 90))
     (property "Footprint" "Capacitor_SMD:C_0402_1005Metric" (id 2) (at 180.34 82.8548 0)
@@
   (symbol (lib_id "Device:C") (at 185.42 100.33 0) (unit 1)
     (in_bom yes) (on_board yes) (fields_autoplaced)
-    (property "Reference" "C33" (id 0) (at 189.23 99.6949 0)
+    (property "Reference" "C34" (id 0) (at 189.23 99.6949 0)
       (effects (font (size 1.27 1.27)) (justify left))
     )
@@
   (symbol (lib_id "Device:C") (at 195.58 100.33 0) (unit 1)
     (in_bom yes) (on_board yes) (fields_autoplaced)
-    (property "Reference" "C34" (id 0) (at 199.39 99.6949 0)
-      (effects (font (size 1.27 1.27)) (justify left))
-    )
+    (property "Reference" "C35" (id 0) (at 199.39 99.6949 0)
+      (effects (font (size 1.27 1.27)) (justify left))
+    )
