File: hardware/RF_front_end/switch.kicad_sch (KiCad schematic)
At the start: 3 parts, among them U2 F2972NEGK

Commit message: Finished front end
Parts:
- renumbered C12 to C13, FB2 to FB3
Changed lines of the file:
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@@
   (symbol (lib_id "power:+3.3V") (at 104.14 43.18 0)
     (in_bom yes) (on_board yes) (fields_autoplaced)
-    (property "Reference" "#PWR013" (id 0) (at 104.14 46.99 0)
+    (property "Reference" "#PWR026" (id 0) (at 104.14 46.99 0)
       (effects (font (size 1.27 1.27)) hide)
     )
@@
   (symbol (lib_id "power:GND") (at 120.65 60.96 0)
     (in_bom yes) (on_board yes) (fields_autoplaced)
-    (property "Reference" "#PWR014" (id 0) (at 120.65 67.31 0)
+    (property "Reference" "#PWR027" (id 0) (at 120.65 67.31 0)
       (effects (font (size 1.27 1.27)) hide)
     )
@@
   (symbol (lib_id "power:GND") (at 124.46 105.41 0)
     (in_bom yes) (on_board yes) (fields_autoplaced)
-    (property "Reference" "#PWR015" (id 0) (at 124.46 111.76 0)
+    (property "Reference" "#PWR028" (id 0) (at 124.46 111.76 0)
       (effects (font (size 1.27 1.27)) hide)
     )
@@
   (symbol (lib_id "Device:FerriteBead_Small") (at 115.57 48.26 90)
     (in_bom yes) (on_board yes) (fields_autoplaced)
-    (property "Reference" "FB2" (id 0) (at 115.57 43.18 90))
+    (property "Reference" "FB3" (id 0) (at 115.57 43.18 90))
     (property "Value" "FerriteBead_Small" (id 1) (at 115.57 45.72 90))
     (property "Footprint" "Inductor_SMD:L_0402_1005Metric" (id 2) (at 115.57 50.038 90)
@@
   (symbol (lib_id "Device:C") (at 120.65 54.61 0)
     (in_bom yes) (on_board yes) (fields_autoplaced)
-    (property "Reference" "C12" (id 0) (at 124.46 53.9749 0)
+    (property "Reference" "C13" (id 0) (at 124.46 53.9749 0)
       (effects (font (size 1.27 1.27)) (justify left))
     )
