File: hardware/RF_front_end/trf37d73.kicad_sch (KiCad schematic)
At the start: 8 parts, among them U1 TRF37D73

Commit message: Finished front end
Parts:
- removed R4: 0, Resistor_SMD:R_0402_1005Metric, symbol Device:R
- renumbered C8 to C14, C9 to C15, C10 to C16, C11 to C17, FB1 to FB4, L2 to L3, U1 to U3
Connections:
- net at C14.1, C15.1, C16.1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: now also L3.1
Changed lines of the file:
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@@
     (stroke (width 0) (type solid) (color 0 0 0 0))
   )
-  (wire (pts (xy 165.1 67.31) (xy 165.1 58.42))
-    (stroke (width 0) (type solid) (color 0 0 0 0))
-  )
-  (wire (pts (xy 165.1 77.47) (xy 165.1 74.93))
+  (wire (pts (xy 165.1 58.42) (xy 165.1 77.47))
     (stroke (width 0) (type solid) (color 0 0 0 0))
   )
@@
   (symbol (lib_id "power:+3.3V") (at 106.68 54.61 0)
     (in_bom yes) (on_board yes) (fields_autoplaced)
-    (property "Reference" "#PWR07" (id 0) (at 106.68 58.42 0)
+    (property "Reference" "#PWR033" (id 0) (at 106.68 58.42 0)
       (effects (font (size 1.27 1.27)) hide)
     )
@@
   (symbol (lib_id "power:GND") (at 123.19 71.12 0)
     (in_bom yes) (on_board yes) (fields_autoplaced)
-    (property "Reference" "#PWR08" (id 0) (at 123.19 77.47 0)
+    (property "Reference" "#PWR034" (id 0) (at 123.19 77.47 0)
       (effects (font (size 1.27 1.27)) hide)
     )
@@
   (symbol (lib_id "power:GND") (at 137.16 114.3 0)
     (in_bom yes) (on_board yes) (fields_autoplaced)
-    (property "Reference" "#PWR09" (id 0) (at 137.16 120.65 0)
+    (property "Reference" "#PWR035" (id 0) (at 137.16 120.65 0)
       (effects (font (size 1.27 1.27)) hide)
     )
@@
   (symbol (lib_id "power:GND") (at 143.51 71.12 0)
     (in_bom yes) (on_board yes) (fields_autoplaced)
-    (property "Reference" "#PWR010" (id 0) (at 143.51 77.47 0)
+    (property "Reference" "#PWR036" (id 0) (at 143.51 77.47 0)
       (effects (font (size 1.27 1.27)) hide)
     )
@@
   (symbol (lib_id "power:GND") (at 151.13 109.22 0)
     (in_bom yes) (on_board yes) (fields_autoplaced)
-    (property "Reference" "#PWR011" (id 0) (at 151.13 115.57 0)
+    (property "Reference" "#PWR037" (id 0) (at 151.13 115.57 0)
       (effects (font (size 1.27 1.27)) hide)
     )
@@
   (symbol (lib_id "power:GND") (at 154.94 71.12 0)
     (in_bom yes) (on_board yes) (fields_autoplaced)
-    (property "Reference" "#PWR012" (id 0) (at 154.94 77.47 0)
+    (property "Reference" "#PWR038" (id 0) (at 154.94 77.47 0)
       (effects (font (size 1.27 1.27)) hide)
     )
@@
   (symbol (lib_id "Device:L") (at 165.1 81.28 0)
     (in_bom yes) (on_board yes)
-    (property "Reference" "L2" (id 0) (at 167.64 80.6449 0)
+    (property "Reference" "L3" (id 0) (at 167.64 80.6449 0)
       (effects (font (size 1.27 1.27)) (justify left))
     )
@@
     (pin "2")
   )
-  (symbol (lib_id "Device:R") (at 165.1 71.12 0)
-    (in_bom yes) (on_board yes) (fields_autoplaced)
-    (property "Reference" "R4" (id 0) (at 167.64 70.4849 0)
-      (effects (font (size 1.27 1.27)) (justify left))
-    )
-    (property "Value" "0" (id 1) (at 167.64 73.0249 0)
-      (effects (font (size 1.27 1.27)) (justify left))
-    )
-    (property "Footprint" "Resistor_SMD:R_0402_1005Metric" (id 2) (at 163.322 71.12 90)
-      (effects (font (size 1.27 1.27)) hide)
-    )
-    (property "Datasheet" "~" (id 3) (at 165.1 71.12 0)
-      (effects (font (size 1.27 1.27)) hide)
-    )
-    (pin "1")
-    (pin "2")
-  )
   (symbol (lib_id "Device:FerriteBead_Small") (at 118.11 58.42 90)
     (in_bom yes) (on_board yes) (fields_autoplaced)
-    (property "Reference" "FB1" (id 0) (at 118.11 53.34 90))
+    (property "Reference" "FB4" (id 0) (at 118.11 53.34 90))
     (property "Value" "FerriteBead_Small" (id 1) (at 118.11 55.88 90))
     (property "Footprint" "Inductor_SMD:L_0402_1005Metric" (id 2) (at 118.11 60.198 90)
@@
   (symbol (lib_id "Device:C") (at 123.19 64.77 0)
     (in_bom yes) (on_board yes) (fields_autoplaced)
-    (property "Reference" "C8" (id 0) (at 127 64.1349 0)
+    (property "Reference" "C14" (id 0) (at 127 64.1349 0)
       (effects (font (size 1.27 1.27)) (justify left))
     )
@@
   (symbol (lib_id "Device:C") (at 143.51 64.77 0)
     (in_bom yes) (on_board yes)
-    (property "Reference" "C9" (id 0) (at 147.32 64.1349 0)
+    (property "Reference" "C15" (id 0) (at 147.32 64.1349 0)
       (effects (font (size 1.27 1.27)) (justify left))
     )
@@
   (symbol (lib_id "Device:C") (at 154.94 64.77 0)
     (in_bom yes) (on_board yes)
-    (property "Reference" "C10" (id 0) (at 158.75 64.1349 0)
+    (property "Reference" "C16" (id 0) (at 158.75 64.1349 0)
       (effects (font (size 1.27 1.27)) (justify left))
     )
@@
   (symbol (lib_id "Device:C") (at 175.26 93.98 90)
     (in_bom yes) (on_board yes) (fields_autoplaced)
-    (property "Reference" "C11" (id 0) (at 175.26 87.63 90))
+    (property "Reference" "C17" (id 0) (at 175.26 87.63 90))
     (property "Value" "100n" (id 1) (at 175.26 90.17 90))
     (property "Footprint" "Capacitor_SMD:C_0402_1005Metric" (id 2) (at 179.07 93.0148 0)
@@
   (symbol (lib_id "RF_WUT:TRF37D73") (at 137.16 93.98 0)
     (in_bom yes) (on_board yes)
-    (property "Reference" "U1" (id 0) (at 139.7 85.09 0))
+    (property "Reference" "U3" (id 0) (at 139.7 85.09 0))
     (property "Value" "TRF37D73" (id 1) (at 143.51 110.49 0))
     (property "Footprint" "Package_SON:WSON-8-1EP_2x2mm_P0.5mm_EP0.9x1.6mm" (id 2) (at 137.16 93.98 0)
