File: hardware/Template_Card/Template_Card.kicad_pcb (KiCad board)
At the start: 4 copper layers, 160 x 100 mm, 9 parts, among them CN1 86093488613755E1LF, J1 Conn_Coaxial, J2 Conn_Coaxial, J3 Conn_Coaxial, U1 24LC024-I/SN, U2 MAX3483ESA+

Commit message: More work on template card
Parts:
- added C10: DNF, Capacitor_SMD:C_0402_1005Metric, F.Cu at (163.6, 68.7)
- added C2: 10u, Capacitor_SMD:C_0603_1608Metric, F.Cu at (186.8, 59.0)
- added C4: 10u, Capacitor_SMD:C_0603_1608Metric, F.Cu at (152.0, 76.2)
- added C5: 100n, Capacitor_SMD:C_0402_1005Metric, F.Cu at (148.8, 67.2)
- added C6: 100n, Capacitor_SMD:C_0402_1005Metric, F.Cu at (148.8, 70.5)
- added C7: 100n, Capacitor_SMD:C_0402_1005Metric, F.Cu at (148.8, 72.0)
- added C9: 100n, Capacitor_SMD:C_0402_1005Metric, F.Cu at (148.8, 73.0)
- added FB1: FerriteBead_Small, Inductor_SMD:L_0603_1608Metric, F.Cu at (141.5, 66.8)
- added J4: USB_B_Micro, Connector_WUT:USB_MicroB_Molex_105133-001_Vertical, F.Cu at (144.8, 66.8)
- added R2: 10k, Resistor_SMD:R_0402_1005Metric, F.Cu at (139.3, 80.3)
- added R3: 4k7, Resistor_SMD:R_0402_1005Metric, F.Cu at (160.7, 66.7)
- added R4: 4k7, Resistor_SMD:R_0402_1005Metric, F.Cu at (155.5, 76.0)
- added R5: 33, Resistor_SMD:R_0402_1005Metric, F.Cu at (148.8, 68.2)
- added R6: 33, Resistor_SMD:R_0402_1005Metric, F.Cu at (148.8, 69.2)
- added U3: MKL26Z64VFT4, Package_DFN_QFN:QFN-48-1EP_7x7mm_P0.5mm_EP5.15x5.15mm, F.Cu at (154.6, 70.3)
- added Y1: 830108178109, Crystal:Crystal_SMD_2016-4Pin_2.0x1.6mm, F.Cu at (143.8, 78.7)
- U1, U2: footprint Package_SO:SO-8_3.9x4.9mm_P1.27mm -> Package_SO:SOIC-8_3.9x4.9mm_P1.27mm
- moved C3 1.00 mm to (185.2, 59.5)
- renumbered C2 to C3
Routing:
- net GND: track 4.25 -> 16.0 mm, vias 4 -> 12
- net +3V3: track 3.58 -> 13.8 mm, vias 1 -> 4
- net /Microcontroller/USB_N: track 0.00 -> 8.98 mm, vias 0 -> 4
- net /Microcontroller/USB_P: track 0.00 -> 7.59 mm, vias 0 -> 4
- net Net-(FB1-Pad1): track 0.00 -> 4.87 mm
- net Net-(C9-Pad1): track 0.00 -> 2.35 mm
- net /Microcontroller/D_P: track 0.00 -> 2.09 mm
- net /Microcontroller/D_N: track 0.00 -> 2.00 mm
- net /RS485_B: track 6.29 -> 7.51 mm
- net /RS485_A: track 6.33 -> 7.34 mm

Commit message: More work on spec
Parts:
- added C8: 100n, Capacitor_SMD:C_0402_1005Metric, F.Cu at (173.5, 73.5)
- moved R2 40.0 mm to (178.5, 72.1), turned to 180 degrees
- moved Y1 33.3 mm to (176.8, 74.3)
- moved R4 26.3 mm to (181.5, 72.0), turned to 90 degrees
- moved R3 22.5 mm to (182.8, 71.5), turned to 90 degrees
- moved C4 18.6 mm to (166.0, 64.0), turned to 180 degrees
- moved U3 17.5 mm to (172.0, 68.5)
- moved C5 17.4 mm to (166.0, 65.5)
- moved C6 17.4 mm to (166.0, 68.8)
- moved C7 17.4 mm to (166.0, 70.3)
- moved C9 17.4 mm to (166.0, 71.3)
- moved FB1 17.4 mm to (158.8, 65.0)
- moved J4 17.4 mm to (162.0, 65.0)
- moved R5 17.4 mm to (166.0, 66.5)
- moved R6 17.4 mm to (166.0, 67.5)
- moved C10 15.1 mm to (178.5, 71.1)
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Connections:
- CN1 pad a11: /SLOTS_EEPROM_3V3 -> unconnected-(CN1-Pada11)
- CN1 pad a12: /SLOTS_EEPROM_WP -> unconnected-(CN1-Pada12)
- CN1 pad a13: unconnected-(CN1-Pada13) -> /SLOTS_EEPROM_3V3
- CN1 pad a14: unconnected-(CN1-Pada14) -> /SLOTS_EEPROM_WP
- CN1 pad a15: /PSU_EEPROM_3V3 -> /PSU_EEPROM_SDA
- CN1 pad b11: /SLOTS_EEPROM_SDA -> unconnected-(CN1-Padb11)
- CN1 pad b12: /SLOTS_EEPROM_SCL -> unconnected-(CN1-Padb12)
- CN1 pad b13: unconnected-(CN1-Padb13) -> /SLOTS_EEPROM_SDA
- CN1 pad b14: unconnected-(CN1-Padb14) -> /SLOTS_EEPROM_SCL
- CN1 pad b15: /PSU_EEPROM_SDA -> /PSU_EEPROM_SCL
- CN1 pad c11: /RS485_B -> unconnected-(CN1-Padc11)
- CN1 pad c12: /RS485_A -> unconnected-(CN1-Padc12)
- CN1 pad c13: unconnected-(CN1-Padc13) -> /RS485_B
- CN1 pad c14: unconnected-(CN1-Padc14) -> /RS485_A
- CN1 pad c15: /PSU_EEPROM_SCL -> /PSU_EEPROM_3V3
- R3 pad 2: /Microcontroller/SCL -> /SLOTS_EEPROM_SCL
- R4 pad 2: /Microcontroller/SDA -> /SLOTS_EEPROM_SDA
- U2 pad 1: unconnected-(U2-Pad1) -> /RX
- U2 pad 2: Net-(U2-Pad2) -> /~{R}/W
- U2 pad 3: Net-(U2-Pad2) -> /~{R}/W
- U2 pad 4: unconnected-(U2-Pad4) -> /TX
- U3 pad 27: /Microcontroller/WP -> /SLOTS_EEPROM_WP
- U3 pad 28: /Microcontroller/~{OVERTEMP} -> unconnected-(U3-Pad28)
- U3 pad 29: /Microcontroller/SCL -> /SLOTS_EEPROM_SCL
- U3 pad 30: /Microcontroller/SDA -> /SLOTS_EEPROM_SDA
- U3 pad 31: /Microcontroller/RX -> /RX
- U3 pad 32: /Microcontroller/TX -> /TX
- U3 pad 33: /Microcontroller/~R~/W -> /~{R}/W
Routing:
- net /SLOTS_EEPROM_SDA: track 0.00 -> 21.8 mm, vias 0 -> 2
- net /SLOTS_EEPROM_WP: track 0.00 -> 21.1 mm, vias 0 -> 1
- net /SLOTS_EEPROM_SCL: track 0.00 -> 19.1 mm
- net GND: track 16.0 -> 27.5 mm, vias 12 -> 25
- net /PSU_EEPROM_3V3: track 16.4 -> 8.43 mm
- net +3V3: track 13.8 -> 21.6 mm, vias 4 -> 9
- net /RX: track 0.00 -> 7.73 mm, vias 0 -> 2
- net /~{R}/W: track 0.00 -> 4.62 mm
- net /TX: track 0.00 -> 4.02 mm
- net Net-(U3-Pad24): track 0.00 -> 3.86 mm
- net /Microcontroller/RESET_B: track 0.00 -> 3.78 mm
- net Net-(U3-Pad25): track 0.00 -> 3.64 mm
- net /PSU_EEPROM_SDA: track 7.04 -> 9.72 mm
- net /PSU_EEPROM_ADDR1: track 10.8 -> 12.5 mm
- net /PSU_EEPROM_ADDR2: track 11.9 -> 13.6 mm
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- added copper zone on In2.Cu, net GND
