File: hardware/Template_Card/Template_Card.kicad_sch (KiCad schematic)
At the start: 9 parts, among them CN1 86093488613755E1LF, J1 Conn_Coaxial, J2 Conn_Coaxial, J3 Conn_Coaxial, U1 24LC024-I/SN, U2 MAX3483ESA+

Commit message: More work on template card
Parts:
- added C2: 10u, Capacitor_SMD:C_0603_1608Metric, symbol Device:C
- U1, U2: footprint Package_SO:SO-8_3.9x4.9mm_P1.27mm -> Package_SO:SOIC-8_3.9x4.9mm_P1.27mm
- renumbered C2 to C3
Connections:
- net +3V3: now also C2.1
- net GND: now also C2.2
Other:
- added sheet Microcontroller (mcu.kicad_sch)

Commit message: More work on spec
Connections:
- net PSU_EEPROM_3V3: now also CN1.c15; no longer CN1.a15
- net PSU_EEPROM_SCL: now also CN1.b15; no longer CN1.c15
- net PSU_EEPROM_SDA: now also CN1.a15; no longer CN1.b15
- net RS485_A: now also CN1.c14; no longer CN1.c12
- net RS485_B: now also CN1.c13; no longer CN1.c11
- net SLOTS_EEPROM_3V3: now also CN1.a13; no longer CN1.a11
- net SLOTS_EEPROM_SCL: now also CN1.b14; no longer CN1.b12
- net SLOTS_EEPROM_SDA: now also CN1.b13; no longer CN1.b11
- net SLOTS_EEPROM_WP: now also CN1.a14; no longer CN1.a12
- net RX: now reaches U2.1 (RO)
- net ~{R}/W: now reaches U2.2 (~{RE}), U2.3 (DE)
- net TX: now reaches U2.4 (DI)
- no-connect marks 6 -> 0
Other:
- sheet Microcontroller ports: added RX, SCL, SDA, TX, WP, ~{R}/W; removed none
Changed lines of the file:
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@@
   (junction (at 200.66 191.77) (diameter 0.9144) (color 0 0 0 0))
   (junction (at 214.63 191.77) (diameter 0.9144) (color 0 0 0 0))
+  (junction (at 215.9 214.63) (diameter 0.9144) (color 0 0 0 0))
   (junction (at 217.17 130.81) (diameter 0.9144) (color 0 0 0 0))
   (junction (at 228.6 165.1) (diameter 0.9144) (color 0 0 0 0))
@@
   (junction (at 354.33 167.64) (diameter 0.9144) (color 0 0 0 0))
   (junction (at 354.33 170.18) (diameter 0.9144) (color 0 0 0 0))
-  (no_connect (at 351.79 66.04))
-  (no_connect (at 351.79 68.58))
-  (no_connect (at 351.79 121.92))
-  (no_connect (at 351.79 124.46))
-  (no_connect (at 351.79 177.8))
-  (no_connect (at 351.79 180.34))
+  (wire (pts (xy 156.21 63.5) (xy 177.8 63.5))
+    (stroke (width 0) (type solid) (color 0 0 0 0))
+  )
+  (wire (pts (xy 156.21 66.04) (xy 177.8 66.04))
+    (stroke (width 0) (type solid) (color 0 0 0 0))
+  )
+  (wire (pts (xy 156.21 68.58) (xy 177.8 68.58))
+    (stroke (width 0) (type solid) (color 0 0 0 0))
+  )
+  (wire (pts (xy 156.21 92.71) (xy 177.8 92.71))
+    (stroke (width 0) (type solid) (color 0 0 0 0))
+  )
+  (wire (pts (xy 156.21 95.25) (xy 177.8 95.25))
+    (stroke (width 0) (type solid) (color 0 0 0 0))
+  )
+  (wire (pts (xy 156.21 97.79) (xy 177.8 97.79))
+    (stroke (width 0) (type solid) (color 0 0 0 0))
+  )
   (wire (pts (xy 195.58 189.23) (xy 195.58 191.77))
     (stroke (width 0) (type solid) (color 0 0 0 0))
@@
     (stroke (width 0) (type solid) (color 0 0 0 0))
   )
+  (wire (pts (xy 205.74 212.09) (xy 218.44 212.09))
+    (stroke (width 0) (type solid) (color 0 0 0 0))
+  )
+  (wire (pts (xy 205.74 214.63) (xy 215.9 214.63))
+    (stroke (width 0) (type solid) (color 0 0 0 0))
+  )
+  (wire (pts (xy 205.74 219.71) (xy 218.44 219.71))
+    (stroke (width 0) (type solid) (color 0 0 0 0))
+  )
   (wire (pts (xy 214.63 191.77) (xy 228.6 191.77))
     (stroke (width 0) (type solid) (color 0 0 0 0))
@@
     (stroke (width 0) (type solid) (color 0 0 0 0))
   )
-  (wire (pts (xy 332.74 60.96) (xy 356.87 60.96))
-    (stroke (width 0) (type solid) (color 0 0 0 0))
-  )
-  (wire (pts (xy 332.74 63.5) (xy 356.87 63.5))
+  (wire (pts (xy 332.74 66.04) (xy 356.87 66.04))
+    (stroke (width 0) (type solid) (color 0 0 0 0))
+  )
+  (wire (pts (xy 332.74 68.58) (xy 356.87 68.58))
     (stroke (width 0) (type solid) (color 0 0 0 0))
   )
@@
     (stroke (width 0) (type solid) (color 0 0 0 0))
   )
-  (wire (pts (xy 332.74 116.84) (xy 356.87 116.84))
-    (stroke (width 0) (type solid) (color 0 0 0 0))
-  )
-  (wire (pts (xy 332.74 119.38) (xy 356.87 119.38))
+  (wire (pts (xy 332.74 121.92) (xy 356.87 121.92))
+    (stroke (width 0) (type solid) (color 0 0 0 0))
+  )
+  (wire (pts (xy 332.74 124.46) (xy 356.87 124.46))
     (stroke (width 0) (type solid) (color 0 0 0 0))
   )
@@
     (stroke (width 0) (type solid) (color 0 0 0 0))
   )
-  (wire (pts (xy 332.74 172.72) (xy 356.87 172.72))
-    (stroke (width 0) (type solid) (color 0 0 0 0))
-  )
-  (wire (pts (xy 332.74 175.26) (xy 356.87 175.26))
+  (wire (pts (xy 332.74 177.8) (xy 356.87 177.8))
+    (stroke (width 0) (type solid) (color 0 0 0 0))
+  )
+  (wire (pts (xy 332.74 180.34) (xy 356.87 180.34))
     (stroke (width 0) (type solid) (color 0 0 0 0))
   )
@@
     (stroke (width 0) (type solid) (color 0 0 0 0))
   )
-  (wire (pts (xy 351.79 66.04) (xy 356.87 66.04))
-    (stroke (width 0) (type solid) (color 0 0 0 0))
-  )
-  (wire (pts (xy 351.79 68.58) (xy 356.87 68.58))
-    (stroke (width 0) (type solid) (color 0 0 0 0))
-  )
-  (wire (pts (xy 351.79 121.92) (xy 356.87 121.92))
-    (stroke (width 0) (type solid) (color 0 0 0 0))
-  )
-  (wire (pts (xy 351.79 124.46) (xy 356.87 124.46))
-    (stroke (width 0) (type solid) (color 0 0 0 0))
-  )
-  (wire (pts (xy 351.79 177.8) (xy 356.87 177.8))
-    (stroke (width 0) (type solid) (color 0 0 0 0))
-  )
-  (wire (pts (xy 351.79 180.34) (xy 356.87 180.34))
-    (stroke (width 0) (type solid) (color 0 0 0 0))
-  )
   (wire (pts (xy 354.33 33.02) (xy 354.33 35.56))
     (stroke (width 0) (type solid) (color 0 0 0 0))
@@
     (stroke (width 0) (type solid) (color 0 0 0 0))
   )
+  (label "TX" (at 177.8 63.5 180)
+    (effects (font (size 1.27 1.27)) (justify right bottom))
+  )
+  (label "RX" (at 177.8 66.04 180)
+    (effects (font (size 1.27 1.27)) (justify right bottom))
+  )
+  (label "~{R}{slash}W" (at 177.8 68.58 180)
+    (effects (font (size 1.27 1.27)) (justify right bottom))
+  )
+  (label "SLOTS_EEPROM_SDA" (at 177.8 92.71 180)
+    (effects (font (size 1.27 1.27)) (justify right bottom))
+  )
+  (label "SLOTS_EEPROM_SCL" (at 177.8 95.25 180)
+    (effects (font (size 1.27 1.27)) (justify right bottom))
+  )
+  (label "SLOTS_EEPROM_WP" (at 177.8 97.79 180)
+    (effects (font (size 1.27 1.27)) (justify right bottom))
+  )
   (label "PSU_EEPROM_3V3" (at 196.85 130.81 0)
     (effects (font (size 1.27 1.27)) (justify left bottom))
@@
   )
   (label "PSU_EEPROM_ADDR2" (at 196.85 158.75 0)
+    (effects (font (size 1.27 1.27)) (justify left bottom))
+  )
+  (label "RX" (at 205.74 212.09 0)
+    (effects (font (size 1.27 1.27)) (justify left bottom))
+  )
+  (label "~{R}{slash}W" (at 205.74 214.63 0)
+    (effects (font (size 1.27 1.27)) (justify left bottom))
+  )
+  (label "TX" (at 205.74 219.71 0)
     (effects (font (size 1.27 1.27)) (justify left bottom))
   )
@@
     (effects (font (size 1.27 1.27)) (justify right bottom))
   )
-  (label "SLOTS_EEPROM_3V3" (at 332.74 60.96 0)
-    (effects (font (size 1.27 1.27)) (justify left bottom))
-  )
-  (label "SLOTS_EEPROM_WP" (at 332.74 63.5 0)
-    (effects (font (size 1.27 1.27)) (justify left bottom))
-  )
-  (label "PSU_EEPROM_3V3" (at 332.74 71.12 0)
+  (label "SLOTS_EEPROM_3V3" (at 332.74 66.04 0)
+    (effects (font (size 1.27 1.27)) (justify left bottom))
+  )
+  (label "SLOTS_EEPROM_WP" (at 332.74 68.58 0)
+    (effects (font (size 1.27 1.27)) (justify left bottom))
+  )
+  (label "PSU_EEPROM_SDA" (at 332.74 71.12 0)
     (effects (font (size 1.27 1.27)) (justify left bottom))
   )
@@
     (effects (font (size 1.27 1.27)) (justify left bottom))
   )
-  (label "SLOTS_EEPROM_SDA" (at 332.74 116.84 0)
-    (effects (font (size 1.27 1.27)) (justify left bottom))
-  )
-  (label "SLOTS_EEPROM_SCL" (at 332.74 119.38 0)
-    (effects (font (size 1.27 1.27)) (justify left bottom))
-  )
-  (label "PSU_EEPROM_SDA" (at 332.74 127 0)
+  (label "SLOTS_EEPROM_SDA" (at 332.74 121.92 0)
+    (effects (font (size 1.27 1.27)) (justify left bottom))
+  )
+  (label "SLOTS_EEPROM_SCL" (at 332.74 124.46 0)
+    (effects (font (size 1.27 1.27)) (justify left bottom))
+  )
+  (label "PSU_EEPROM_SCL" (at 332.74 127 0)
     (effects (font (size 1.27 1.27)) (justify left bottom))
   )
@@
     (effects (font (size 1.27 1.27)) (justify left bottom))
   )
-  (label "RS485_B" (at 332.74 172.72 0)
-    (effects (font (size 1.27 1.27)) (justify left bottom))
-  )
-  (label "RS485_A" (at 332.74 175.26 0)
-    (effects (font (size 1.27 1.27)) (justify left bottom))
-  )
-  (label "PSU_EEPROM_SCL" (at 332.74 182.88 0)
+  (label "RS485_B" (at 332.74 177.8 0)
+    (effects (font (size 1.27 1.27)) (justify left bottom))
+  )
+  (label "RS485_A" (at 332.74 180.34 0)
+    (effects (font (size 1.27 1.27)) (justify left bottom))
+  )
+  (label "PSU_EEPROM_3V3" (at 332.74 182.88 0)
     (effects (font (size 1.27 1.27)) (justify left bottom))
   )
@@
       (effects (font (size 1.27 1.27)) (justify left top))
     )
+    (pin "TX" output (at 156.21 63.5 0)
+      (effects (font (size 1.27 1.27)) (justify right))
+    )
+    (pin "RX" input (at 156.21 66.04 0)
+      (effects (font (size 1.27 1.27)) (justify right))
+    )
+    (pin "SDA" bidirectional (at 156.21 92.71 0)
+      (effects (font (size 1.27 1.27)) (justify right))
+    )
+    (pin "SCL" output (at 156.21 95.25 0)
+      (effects (font (size 1.27 1.27)) (justify right))
+    )
+    (pin "~{R}{slash}W" output (at 156.21 68.58 0)
+      (effects (font (size 1.27 1.27)) (justify right))
+    )
+    (pin "WP" input (at 156.21 97.79 0)
+      (effects (font (size 1.27 1.27)) (justify right))
+    )
   )
   (sheet_instances
@@
       (reference "C7") (unit 1) (value "100n") (footprint "Capacitor_SMD:C_0402_1005Metric")
     )
+    (path "/6c3b16c4-1007-44f2-988d-7aebc0401692/c58db099-f401-4541-ba3f-fd24183e5e43"
+      (reference "C8") (unit 1) (value "100n") (footprint "Capacitor_SMD:C_0402_1005Metric")
+    )
     (path "/6c3b16c4-1007-44f2-988d-7aebc0401692/8197e698-4c2e-409c-8aad-f231ae7fd6ed"
