File: hardware/Template_Card/mcu.kicad_sch (KiCad schematic)
At the start: 15 parts, among them J4 USB_B_Micro, U3 MKL26Z64VFT4, Y1 830108178109

Commit message: More work on spec
Parts:
- added C8: 100n, Capacitor_SMD:C_0402_1005Metric, symbol Device:C
Connections:
- net +3V3: now also C8.1
- net GND: now also C8.2
- net ~R~/W renamed ~{R}/W
- net ~{OVERTEMP}: no longer names the net of U3.28 (PTB1)
Changed lines of the file:
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@@
   (junction (at 170.18 78.74) (diameter 0.9144) (color 0 0 0 0))
   (junction (at 181.61 67.31) (diameter 0.9144) (color 0 0 0 0))
+  (junction (at 181.61 78.74) (diameter 0.9144) (color 0 0 0 0))
+  (junction (at 193.04 67.31) (diameter 0.9144) (color 0 0 0 0))
   (junction (at 207.01 67.31) (diameter 0.9144) (color 0 0 0 0))
   (junction (at 212.09 67.31) (diameter 0.9144) (color 0 0 0 0))
@@
     (stroke (width 0) (type solid) (color 0 0 0 0))
   )
-  (wire (pts (xy 167.64 137.16) (xy 184.15 137.16))
-    (stroke (width 0) (type solid) (color 0 0 0 0))
-  )
   (wire (pts (xy 167.64 144.78) (xy 184.15 144.78))
     (stroke (width 0) (type solid) (color 0 0 0 0))
@@
     (stroke (width 0) (type solid) (color 0 0 0 0))
   )
-  (wire (pts (xy 181.61 67.31) (xy 207.01 67.31))
+  (wire (pts (xy 181.61 67.31) (xy 193.04 67.31))
     (stroke (width 0) (type solid) (color 0 0 0 0))
   )
@@
     (stroke (width 0) (type solid) (color 0 0 0 0))
   )
+  (wire (pts (xy 181.61 78.74) (xy 193.04 78.74))
+    (stroke (width 0) (type solid) (color 0 0 0 0))
+  )
   (wire (pts (xy 184.15 127) (xy 172.72 127))
     (stroke (width 0) (type solid) (color 0 0 0 0))
   )
+  (wire (pts (xy 193.04 67.31) (xy 193.04 69.85))
+    (stroke (width 0) (type solid) (color 0 0 0 0))
+  )
+  (wire (pts (xy 193.04 67.31) (xy 207.01 67.31))
+    (stroke (width 0) (type solid) (color 0 0 0 0))
+  )
+  (wire (pts (xy 193.04 77.47) (xy 193.04 78.74))
+    (stroke (width 0) (type solid) (color 0 0 0 0))
+  )
   (wire (pts (xy 207.01 67.31) (xy 207.01 86.36))
     (stroke (width 0) (type solid) (color 0 0 0 0))
@@
     (effects (font (size 1.27 1.27)) (justify left bottom))
   )
-  (label "SCL" (at 129.54 147.32 0)
-    (effects (font (size 1.27 1.27)) (justify left bottom))
-  )
-  (label "SDA" (at 129.54 149.86 0)
-    (effects (font (size 1.27 1.27)) (justify left bottom))
-  )
-  (label "WP" (at 167.64 134.62 0)
-    (effects (font (size 1.27 1.27)) (justify left bottom))
-  )
-  (label "~{OVERTEMP}" (at 167.64 137.16 0)
-    (effects (font (size 1.27 1.27)) (justify left bottom))
-  )
-  (label "RX" (at 167.64 144.78 0)
-    (effects (font (size 1.27 1.27)) (justify left bottom))
-  )
-  (label "TX" (at 167.64 147.32 0)
-    (effects (font (size 1.27 1.27)) (justify left bottom))
-  )
   (label "PTA0" (at 168.91 104.14 0)
     (effects (font (size 1.27 1.27)) (justify left bottom))
@@
     (effects (font (size 1.27 1.27)) (justify left bottom))
   )
-  (label "~R~{slash}W" (at 262.89 104.14 180)
-    (effects (font (size 1.27 1.27)) (justify right bottom))
-  )
   (label "SPARE_9" (at 262.89 106.68 180)
     (effects (font (size 1.27 1.27)) (justify right bottom))
@@
   (label "LED_RX" (at 262.89 154.94 180)
     (effects (font (size 1.27 1.27)) (justify right bottom))
+  )
+  (hierarchical_label "SCL" (shape output) (at 129.54 147.32 180)
+    (effects (font (size 1.27 1.27)) (justify right))
+  )
+  (hierarchical_label "SDA" (shape bidirectional) (at 129.54 149.86 180)
+    (effects (font (size 1.27 1.27)) (justify right))
+  )
+  (hierarchical_label "WP" (shape input) (at 167.64 134.62 180)
+    (effects (font (size 1.27 1.27)) (justify right))
+  )
+  (hierarchical_label "RX" (shape input) (at 167.64 144.78 180)
+    (effects (font (size 1.27 1.27)) (justify right))
+  )
+  (hierarchical_label "TX" (shape output) (at 167.64 147.32 180)
+    (effects (font (size 1.27 1.27)) (justify right))
+  )
+  (hierarchical_label "~{R}{slash}W" (shape output) (at 262.89 104.14 0)
+    (effects (font (size 1.27 1.27)) (justify left))
   )
   (symbol (lib_id "power:+3.3V") (at 127 110.49 0) (unit 1)
@@
       (effects (font (size 1.27 1.27)) hide)
     )
+    (pin "1")
+    (pin "2")
+  )
+  (symbol (lib_id "Device:C") (at 193.04 73.66 0) (unit 1)
+    (in_bom yes) (on_board yes) (fields_autoplaced)
+    (property "Reference" "C8" (id 0) (at 196.85 73.0249 0)
+      (effects (font (size 1.27 1.27)) (justify left))
+    )
+    (property "Value" "100n" (id 1) (at 196.85 75.5649 0)
+      (effects (font (size 1.27 1.27)) (justify left))
+    )
+    (property "Footprint" "Capacitor_SMD:C_0402_1005Metric" (id 2) (at 194.0052 77.47 0)
+      (effects (font (size 1.27 1.27)) hide)
+    )
+    (property "Datasheet" "~" (id 3) (at 193.04 73.66 0)
+      (effects (font (size 1.27 1.27)) hide)
+    )
