File: hardware/soldering_test/soldering_test.kicad_sch (KiCad schematic)
At the start: 2 parts, among them CN1 FMC_Mezzanine, U1 Xilinx_Kria_SM-K26-XCL2GC_SOM

Commit message: Started on FMC card template
Parts:
- added M1: Logo_10mmx10mm, Misc_WUT:Logo_10mmx10mm, symbol Misc_WUT:Logo_10mmx10mm
Changed lines of the file:
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@@
     (stroke (width 0) (type default) (color 0 0 0 0))
+  )
+  (symbol (lib_id "Misc_WUT:Logo_10mmx10mm") (at 102.87 262.89 0) (unit 1)
+    (in_bom no) (on_board yes) (fields_autoplaced)
+    (property "Reference" "M1" (id 0) (at 103.505 261.9815 0)
+      (effects (font (size 1.27 1.27)) (justify left))
+    )
+    (property "Value" "Logo_10mmx10mm" (id 1) (at 103.505 264.7566 0)
+      (effects (font (size 1.27 1.27)) (justify left))
+    )
+    (property "Footprint" "Misc_WUT:Logo_10mmx10mm" (id 2) (at 102.87 262.89 0)
+      (effects (font (size 1.27 1.27)) hide)
+    )
+    (property "Datasheet" "" (id 3) (at 102.87 262.89 0)
+      (effects (font (size 1.27 1.27)) hide)
+    )
   )
   (symbol (lib_id "power:GND") (at 34.29 264.16 0) (unit 1)
@@
       (reference "CN1") (unit 2) (value "FMC_Mezzanine") (footprint "Connector_WUT:Samtec_FMC_ASP-134604-01_4x40_Vertical")
     )
+    (path "/0f710616-9e8f-4839-871b-47ab2498ee4f"
+      (reference "M1") (unit 1) (value "Logo_10mmx10mm") (footprint "Misc_WUT:Logo_10mmx10mm")
+    )
     (path "/71b592a8-884c-477b-b9ae-af51ee5a5cac"
