File: hardware/RF_FMC/fmcConnector.kicad_sch (KiCad schematic)
At the start: 42 parts, among them CN1 FMC_Mezzanine, M1 Logo_10mmx10mm, U1 24LC02BT-I/MNY, U2 LM73100RPWR, U3 LM73100RPWR, U4 LM73100RPWR

Commit message: Started on ADC layout
Parts:
- renumbered R9 to R10, R10 to R11, R11 to R12, R12 to R13, R13 to R14, R14 to R15, R15 to R16, R16 to R17, R17 to R18, R1 to R2, R2 to R3, R3 to R4, R4 to R5, R5 to R6, R6 to R7, R7 to R8, R8 to R9
Changed lines of the file:
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@@
   (symbol (lib_id "Device:R") (at 34.29 168.91 0) (unit 1)
     (in_bom yes) (on_board yes) (fields_autoplaced)
-    (property "Reference" "R1" (id 0) (at 36.0681 168.0015 0)
+    (property "Reference" "R2" (id 0) (at 36.0681 168.0015 0)
       (effects (font (size 1.27 1.27)) (justify left))
     )
@@
   (symbol (lib_id "Device:R") (at 34.29 179.07 0) (unit 1)
     (in_bom yes) (on_board yes) (fields_autoplaced)
-    (property "Reference" "R2" (id 0) (at 36.0681 178.1615 0)
+    (property "Reference" "R3" (id 0) (at 36.0681 178.1615 0)
       (effects (font (size 1.27 1.27)) (justify left))
     )
@@
   (symbol (lib_id "Device:R") (at 83.82 161.29 0) (unit 1)
     (in_bom yes) (on_board yes) (fields_autoplaced)
-    (property "Reference" "R3" (id 0) (at 85.5981 160.3815 0)
+    (property "Reference" "R4" (id 0) (at 85.5981 160.3815 0)
       (effects (font (size 1.27 1.27)) (justify left))
     )
@@
   (symbol (lib_id "Device:R") (at 92.71 161.29 0) (unit 1)
     (in_bom yes) (on_board yes) (fields_autoplaced)
-    (property "Reference" "R4" (id 0) (at 94.4881 160.3815 0)
+    (property "Reference" "R5" (id 0) (at 94.4881 160.3815 0)
       (effects (font (size 1.27 1.27)) (justify left))
     )
@@
   (symbol (lib_id "Device:R") (at 138.43 163.83 0) (unit 1)
     (in_bom yes) (on_board yes) (fields_autoplaced)
-    (property "Reference" "R5" (id 0) (at 140.2081 162.9215 0)
+    (property "Reference" "R6" (id 0) (at 140.2081 162.9215 0)
       (effects (font (size 1.27 1.27)) (justify left))
     )
@@
   (symbol (lib_id "Device:R") (at 193.04 44.45 90) (unit 1)
     (in_bom yes) (on_board yes) (fields_autoplaced)
-    (property "Reference" "R6" (id 0) (at 193.04 39.4674 90))
+    (property "Reference" "R7" (id 0) (at 193.04 39.4674 90))
     (property "Value" "1k" (id 1) (at 193.04 42.2425 90))
     (property "Footprint" "Resistor_SMD:R_0402_1005Metric" (id 2) (at 193.04 46.228 90)
@@
   (symbol (lib_id "Device:R") (at 193.04 91.44 90) (unit 1)
     (in_bom yes) (on_board yes) (fields_autoplaced)
-    (property "Reference" "R7" (id 0) (at 193.04 86.4574 90))
+    (property "Reference" "R8" (id 0) (at 193.04 86.4574 90))
     (property "Value" "1k" (id 1) (at 193.04 89.2325 90))
     (property "Footprint" "Resistor_SMD:R_0402_1005Metric" (id 2) (at 193.04 93.218 90)
@@
   (symbol (lib_id "Device:R") (at 193.04 138.43 90) (unit 1)
     (in_bom yes) (on_board yes) (fields_autoplaced)
-    (property "Reference" "R8" (id 0) (at 193.04 133.4474 90))
+    (property "Reference" "R9" (id 0) (at 193.04 133.4474 90))
     (property "Value" "1k" (id 1) (at 193.04 136.2225 90))
     (property "Footprint" "Resistor_SMD:R_0402_1005Metric" (id 2) (at 193.04 140.208 90)
@@
   (symbol (lib_id "Device:R") (at 208.28 50.8 0) (unit 1)
     (in_bom yes) (on_board yes) (fields_autoplaced)
-    (property "Reference" "R9" (id 0) (at 210.0581 49.8915 0)
+    (property "Reference" "R10" (id 0) (at 210.0581 49.8915 0)
       (effects (font (size 1.27 1.27)) (justify left))
     )
@@
   (symbol (lib_id "Device:R") (at 208.28 97.79 0) (unit 1)
     (in_bom yes) (on_board yes) (fields_autoplaced)
-    (property "Reference" "R10" (id 0) (at 210.0581 96.8815 0)
+    (property "Reference" "R11" (id 0) (at 210.0581 96.8815 0)
       (effects (font (size 1.27 1.27)) (justify left))
     )
@@
   (symbol (lib_id "Device:R") (at 208.28 144.78 0) (unit 1)
     (in_bom yes) (on_board yes) (fields_autoplaced)
-    (property "Reference" "R11" (id 0) (at 210.0581 143.8715 0)
+    (property "Reference" "R12" (id 0) (at 210.0581 143.8715 0)
       (effects (font (size 1.27 1.27)) (justify left))
     )
@@
   (symbol (lib_id "Device:R") (at 218.44 43.18 0) (unit 1)
     (in_bom yes) (on_board yes) (fields_autoplaced)
-    (property "Reference" "R12" (id 0) (at 220.2181 42.2715 0)
+    (property "Reference" "R13" (id 0) (at 220.2181 42.2715 0)
       (effects (font (size 1.27 1.27)) (justify left))
     )
@@
   (symbol (lib_id "Device:R") (at 218.44 90.17 0) (unit 1)
     (in_bom yes) (on_board yes) (fields_autoplaced)
-    (property "Reference" "R13" (id 0) (at 220.2181 89.2615 0)
+    (property "Reference" "R14" (id 0) (at 220.2181 89.2615 0)
       (effects (font (size 1.27 1.27)) (justify left))
     )
@@
   (symbol (lib_id "Device:R") (at 218.44 137.16 0) (unit 1)
     (in_bom yes) (on_board yes) (fields_autoplaced)
-    (property "Reference" "R14" (id 0) (at 220.2181 136.2515 0)
+    (property "Reference" "R15" (id 0) (at 220.2181 136.2515 0)
       (effects (font (size 1.27 1.27)) (justify left))
     )
@@
   (symbol (lib_id "Device:R") (at 255.27 44.45 0) (unit 1)
     (in_bom yes) (on_board yes) (fields_autoplaced)
-    (property "Reference" "R15" (id 0) (at 257.0481 43.5415 0)
+    (property "Reference" "R16" (id 0) (at 257.0481 43.5415 0)
       (effects (font (size 1.27 1.27)) (justify left))
     )
@@
   (symbol (lib_id "Device:R") (at 255.27 91.44 0) (unit 1)
     (in_bom yes) (on_board yes) (fields_autoplaced)
-    (property "Reference" "R16" (id 0) (at 257.0481 90.5315 0)
+    (property "Reference" "R17" (id 0) (at 257.0481 90.5315 0)
       (effects (font (size 1.27 1.27)) (justify left))
     )
@@
   (symbol (lib_id "Device:R") (at 255.27 138.43 0) (unit 1)
     (in_bom yes) (on_board yes) (fields_autoplaced)
-    (property "Reference" "R17" (id 0) (at 257.0481 137.5215 0)
-      (effects (font (size 1.27 1.27)) (justify left))
-    )
+    (property "Reference" "R18" (id 0) (at 257.0481 137.5215 0)
+      (effects (font (size 1.27 1.27)) (justify left))
+    )
